File: schematic/AutoDischarger/discharge_control.kicad_sch (KiCad schematic)
At the start: 28 parts, among them Q1 2N7002_HAMR, Q10 2N7002_HAMR, Q11 2N7002_HAMR, Q2 2N7002_HAMR, Q3 2N7002_HAMR, Q4 2N7002_HAMR, Q5 2N7002_HAMR, Q6 2N7002_HAMR, Q7 2N7002_HAMR, Q8 2N7002_HAMR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

Commit message: Some schematic fixes and assigned footprints.
Parts:
- Q1, Q10, Q11, Q2, Q3, Q4, Q5, Q6, Q7, Q8, Q9: footprint 2N7002HAMR -> SamacSys_Parts:2N7002HAMR
- R32, R33, R34, R35, R36, R37, R38, R39, R40, R41, R42: footprint (none) -> Resistor_SMD:R_0603_1608Metric
- R43, R44, R45, R46, R47, R48: footprint (none) -> Resistor_SMD:R_1206_3216Metric
Other:
- note added: "2S"
- note added: "3S"
- note added: "4S"
- note added: "5S"
- note added: "6S"
- company: Quantum Embedded System -> Quantum Embedded Systems

Commit message: Some schematic and footprint fixes
Parts:
- Q1, Q10, Q11, Q2, Q3, Q4, Q5, Q6, Q7, Q8, Q9: footprint SamacSys_Parts:2N7002HAMR -> Package_TO_SOT_SMD:SOT-23
Changed lines of the file:
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@@
       (effects (font (size 1.27 1.27)) (justify left))
     )
-    (property "Footprint" "SamacSys_Parts:2N7002HAMR" (id 2) (at 64.77 149.86 0)
+    (property "Footprint" "Package_TO_SOT_SMD:SOT-23" (id 2) (at 64.77 149.86 0)
       (effects (font (size 1.27 1.27)) (justify left) hide)
     )
@@
       (effects (font (size 1.27 1.27)) (justify left))
     )
-    (property "Footprint" "SamacSys_Parts:2N7002HAMR" (id 2) (at 114.935 70.485 0)
+    (property "Footprint" "Package_TO_SOT_SMD:SOT-23" (id 2) (at 114.935 70.485 0)
       (effects (font (size 1.27 1.27)) (justify left) hide)
     )
@@
       (effects (font (size 1.27 1.27)) (justify left))
     )
-    (property "Footprint" "SamacSys_Parts:2N7002HAMR" (id 2) (at 114.935 174.625 0)
+    (property "Footprint" "Package_TO_SOT_SMD:SOT-23" (id 2) (at 114.935 174.625 0)
       (effects (font (size 1.27 1.27)) (justify left) hide)
     )
@@
       (effects (font (size 1.27 1.27)) (justify left))
     )
-    (property "Footprint" "SamacSys_Parts:2N7002HAMR" (id 2) (at 114.935 95.25 0)
+    (property "Footprint" "Package_TO_SOT_SMD:SOT-23" (id 2) (at 114.935 95.25 0)
       (effects (font (size 1.27 1.27)) (justify left) hide)
     )
@@
       (effects (font (size 1.27 1.27)) (justify left))
     )
-    (property "Footprint" "SamacSys_Parts:2N7002HAMR" (id 2) (at 114.935 44.45 0)
+    (property "Footprint" "Package_TO_SOT_SMD:SOT-23" (id 2) (at 114.935 44.45 0)
       (effects (font (size 1.27 1.27)) (justify left) hide)
     )
@@
       (effects (font (size 1.27 1.27)) (justify left))
     )
-    (property "Footprint" "SamacSys_Parts:2N7002HAMR" (id 2) (at 64.77 71.12 0)
+    (property "Footprint" "Package_TO_SOT_SMD:SOT-23" (id 2) (at 64.77 71.12 0)
       (effects (font (size 1.27 1.27)) (justify left) hide)
     )
@@
       (effects (font (size 1.27 1.27)) (justify left))
     )
-    (property "Footprint" "SamacSys_Parts:2N7002HAMR" (id 2) (at 64.77 95.885 0)
+    (property "Footprint" "Package_TO_SOT_SMD:SOT-23" (id 2) (at 64.77 95.885 0)
       (effects (font (size 1.27 1.27)) (justify left) hide)
     )
@@
       (effects (font (size 1.27 1.27)) (justify left))
     )
-    (property "Footprint" "SamacSys_Parts:2N7002HAMR" (id 2) (at 64.77 45.72 0)
+    (property "Footprint" "Package_TO_SOT_SMD:SOT-23" (id 2) (at 64.77 45.72 0)
       (effects (font (size 1.27 1.27)) (justify left) hide)
     )
@@
       (effects (font (size 1.27 1.27)) (justify left))
     )
-    (property "Footprint" "SamacSys_Parts:2N7002HAMR" (id 2) (at 114.935 123.19 0)
+    (property "Footprint" "Package_TO_SOT_SMD:SOT-23" (id 2) (at 114.935 123.19 0)
       (effects (font (size 1.27 1.27)) (justify left) hide)
     )
@@
       (effects (font (size 1.27 1.27)) (justify left))
     )
-    (property "Footprint" "SamacSys_Parts:2N7002HAMR" (id 2) (at 114.935 149.225 0)
+    (property "Footprint" "Package_TO_SOT_SMD:SOT-23" (id 2) (at 114.935 149.225 0)
       (effects (font (size 1.27 1.27)) (justify left) hide)
     )
@@
       (effects (font (size 1.27 1.27)) (justify left))
     )
-    (property "Footprint" "SamacSys_Parts:2N7002HAMR" (id 2) (at 64.77 123.825 0)
-      (effects (font (size 1.27 1.27)) (justify left) hide)
-    )
+    (property "Footprint" "Package_TO_SOT_SMD:SOT-23" (id 2) (at 64.77 123.825 0)
+      (effects (font (size 1.27 1.27)) (justify left) hide)
+    )

Commit message: Updated for 18R 1W 2512 resistors
Parts:
- R43, R44, R45, R46, R47, R48: value 120R -> 18R; footprint Resistor_SMD:R_1206_3216Metric -> Resistor_SMD:R_2512_6332Metric
Other:
- note added: "Discharge resistors (R43,R44,R45,R46,R47,R48) should be at least 1W"
Changed lines of the file:
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@@
     (effects (font (size 4 4)) (justify left bottom))
+  )
+  (text "Discharge resistors \n(R43,R44,R45,R46,R47,R48) \nshould be at least 1W "
+    (at 158.115 119.38 0)
+    (effects (font (size 1.27 1.27)) (justify left bottom))
   )
   (text "6S" (at 135.89 40.64 0)
@@
     (in_bom yes) (on_board yes) (fields_autoplaced)
     (property "Reference" "R45" (id 0) (at 137.16 76.9325 90))
-    (property "Value" "120R" (id 1) (at 137.16 79.7076 90))
-    (property "Footprint" "Resistor_SMD:R_1206_3216Metric" (id 2) (at 137.16 83.693 90)
+    (property "Value" "18R" (id 1) (at 137.16 79.7076 90))
+    (property "Footprint" "Resistor_SMD:R_2512_6332Metric" (id 2) (at 137.16 83.693 90)
       (effects (font (size 1.27 1.27)) hide)
     )
@@
     (in_bom yes) (on_board yes) (fields_autoplaced)
     (property "Reference" "R48" (id 0) (at 137.16 155.6725 90))
-    (property "Value" "120R" (id 1) (at 137.16 158.4476 90))
-    (property "Footprint" "Resistor_SMD:R_1206_3216Metric" (id 2) (at 137.16 162.433 90)
+    (property "Value" "18R" (id 1) (at 137.16 158.4476 90))
+    (property "Footprint" "Resistor_SMD:R_2512_6332Metric" (id 2) (at 137.16 162.433 90)
       (effects (font (size 1.27 1.27)) hide)
     )
@@
     (in_bom yes) (on_board yes) (fields_autoplaced)
     (property "Reference" "R43" (id 0) (at 136.525 21.0525 90))
-    (property "Value" "120R" (id 1) (at 136.525 23.8276 90))
-    (property "Footprint" "Resistor_SMD:R_1206_3216Metric" (id 2) (at 136.525 27.813 90)
+    (property "Value" "18R" (id 1) (at 136.525 23.8276 90))
+    (property "Footprint" "Resistor_SMD:R_2512_6332Metric" (id 2) (at 136.525 27.813 90)
       (effects (font (size 1.27 1.27)) hide)
     )
@@
     (in_bom yes) (on_board yes) (fields_autoplaced)
     (property "Reference" "R44" (id 0) (at 137.16 51.5325 90))
-    (property "Value" "120R" (id 1) (at 137.16 54.3076 90))
-    (property "Footprint" "Resistor_SMD:R_1206_3216Metric" (id 2) (at 137.16 58.293 90)
+    (property "Value" "18R" (id 1) (at 137.16 54.3076 90))
+    (property "Footprint" "Resistor_SMD:R_2512_6332Metric" (id 2) (at 137.16 58.293 90)
       (effects (font (size 1.27 1.27)) hide)
     )
@@
     (in_bom yes) (on_board yes) (fields_autoplaced)
     (property "Reference" "R47" (id 0) (at 137.16 130.9075 90))
-    (property "Value" "120R" (id 1) (at 137.16 133.6826 90))
-    (property "Footprint" "Resistor_SMD:R_1206_3216Metric" (id 2) (at 137.16 137.668 90)
+    (property "Value" "18R" (id 1) (at 137.16 133.6826 90))
+    (property "Footprint" "Resistor_SMD:R_2512_6332Metric" (id 2) (at 137.16 137.668 90)
       (effects (font (size 1.27 1.27)) hide)
     )
@@
     (in_bom yes) (on_board yes) (fields_autoplaced)
     (property "Reference" "R46" (id 0) (at 137.16 104.2375 90))
-    (property "Value" "120R" (id 1) (at 137.16 107.0126 90))
-    (property "Footprint" "Resistor_SMD:R_1206_3216Metric" (id 2) (at 137.16 110.998 90)
-      (effects (font (size 1.27 1.27)) hide)
-    )
+    (property "Value" "18R" (id 1) (at 137.16 107.0126 90))
+    (property "Footprint" "Resistor_SMD:R_2512_6332Metric" (id 2) (at 137.16 110.998 90)
+      (effects (font (size 1.27 1.27)) hide)
+    )
